File: PCB/RMOC-SC/RMOC-SC/RMOC-SC.kicad_sch (KiCad schematic)
At the start: 39 parts, among them J1 Conn_01x02_Pin, Q1 TIC106, Q2 TIC106, U1 ACS712xLCTR-20A, U2 PC817, U3 MOC3021M, U4 MOC3021M, U5 ESP32-DEVKITV1-30PIN, U6 5V700mA 3.5W

Commit message: Simulación en 12V + Dualidad 12V-220V en PCB
Parts:
- added C4: 100n, Capacitor_THT:C_Disc_D5.0mm_W2.5mm_P5.00mm, symbol Device:C
- added J2, J3, J4, J5, J8: Conn_01x03_Pin, Connector_PinHeader_2.54mm:PinHeader_1x03_P2.54mm_Vertical, symbol Connector:Conn_01x03_Pin
- added R1: 1K5, symbol Device:R_US
- added R15: 2K, symbol Device:R_US
- added R16: 1K, symbol Device:R_US
- added R6: 220, symbol Device:R_US
- added R7: 2K2, symbol Device:R_US
- added R9: 18K, symbol Device:R_US
- J1: footprint Connector:Tag-Connect_TC2030-IDC-NL_2x03_P1.27mm_Vertical -> Connector_PinHeader_2.54mm:PinHeader_1x02_P2.54mm_Vertical
- R12: renamed from R6; value 47K -> 10K
- R5: renamed from R7; value 470 -> 2K2
- R8: value 470 -> 220
- TP1, TP2, TP3: footprint (none) -> Connector_PinHeader_2.54mm:PinHeader_1x01_P2.54mm_Vertical
- TP10: renamed from TP8; footprint (none) -> Connector_PinHeader_2.54mm:PinHeader_1x01_P2.54mm_Vertical
- TP4: renamed from TP9; footprint (none) -> Connector_PinHeader_2.54mm:PinHeader_1x01_P2.54mm_Vertical
- TP5: renamed from TP10; footprint (none) -> Connector_PinHeader_2.54mm:PinHeader_1x01_P2.54mm_Vertical
- TP6: renamed from TP4; footprint (none) -> Connector_PinHeader_2.54mm:PinHeader_1x01_P2.54mm_Vertical
- TP7: renamed from TP5; footprint (none) -> Connector_PinHeader_2.54mm:PinHeader_1x01_P2.54mm_Vertical
- TP8: renamed from TP6; footprint (none) -> Connector_PinHeader_2.54mm:PinHeader_1x01_P2.54mm_Vertical
- TP9: renamed from TP7; footprint (none) -> Connector_PinHeader_2.54mm:PinHeader_1x01_P2.54mm_Vertical
- renumbered C2 to C1, C3 to C2, C1 to C3, D3 to D1, D4 to D2, D5 to D3, D2 to D4, D1 to D5, R3 to R10, R4 to R11, R1 to R13, R2 to R14, R5 to R2, R9 to R3, R10 to R4, U6 to U1, U5 to U2, U4 to U3, U3 to U4, U2 to U5, U1 to U6
Connections:
- net +5V: now also C4.1
- net GND: now also C4.2, J8.3 (Pin_3), R15.2
- net IP-: now also J8.2 (Pin_2); no longer C2.1, R13.2, R14.1
- net LINE: now also R1.1
- net Vadc: now also TP8.1, J3.2 (Pin_2); no longer R10.2
- net Valpha: now also TP10.1
- net Vdisp1: now also TP6.1, J4.2 (Pin_2); no longer R5.2
- net Vdisp2: now also TP7.1, J5.2 (Pin_2); no longer R8.2
- net Viout: now also TP9.1, R15.1, R16.2; no longer U6.7 (VIOUT)
- net Vout: now also R9.1
- net at R5.1, U4.4: now also R6.1
- net at R8.1, U3.4: now also R7.1
- net at D5.1 (K), U5.1: now also J2.2 (Pin_2); no longer R2.2
- new net: R16.1, U6.7 (VIOUT)
- new net Radc_12: J3.3 (Pin_3), R9.2
- new net Radc_220: J3.1 (Pin_1), R10.2
- new net Rdisp1_12: J4.3 (Pin_3), R6.2
- new net Rdisp1_220: J4.1 (Pin_1), R5.2
- new net Rdisp2_12: J5.3 (Pin_3), R8.2
- new net Rdisp2_220: J5.1 (Pin_1), R7.2
- new net Ropto_12: J2.3 (Pin_3), R1.2
- new net Ropto_220: J2.1 (Pin_1), R2.2
- new net V_1.65: C2.1, J8.1 (Pin_1), R13.2, R14.1
Other:
- note added: "J2 selector de R de entrada al optoacoplador"
- note added: "J3 selector de R de sensado"
- note added: "J4 y J5 selector de R de disparo"
- note added: "J8 selector de Tierra Virtual (1.65V - 0V)"
- note added: "Valores de R para 220V R's para testear a 10/12V Testpoints Fuente HLK-PM01? interlock pcb?"
- note removed: "R's para testear a 10/12V Testpoints Fuente HLK-PM01? interlock pcb?"
- moved on the sheet: C1, C2, C3, D3, D4, D5, R10, R11, R12, R13, R14, R2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

Commit message: Inicio de PCB
Parts:
- added R17: 12K, Resistor_THT:R_Axial_DIN0614_L14.3mm_D5.7mm_P20.32mm_Horizontal, symbol Device:R_US
- J1: footprint Connector_PinHeader_2.54mm:PinHeader_1x02_P2.54mm_Vertical -> WX-DC12003:Conn_220_tipo8
- R1, R10, R11, R12, R13, R14, R15, R16, R3, R4, R5, R6, R7, R8, R9: footprint (none) -> Resistor_THT:R_Axial_DIN0309_L9.0mm_D3.2mm_P12.70mm_Horizontal
- R2: value 22K -> 10K; footprint (none) -> Resistor_THT:R_Axial_DIN0614_L14.3mm_D5.7mm_P20.32mm_Horizontal
- RL1: footprint (none) -> TerminalBlock_Altech:Altech_AK100_1x02_P5.00mm
- RV1: footprint Package_SO:TSSOP-20_4.4x6.5mm_P0.65mm -> Potentiometer_THT:Potentiometer_Piher_PC-16_Single_Horizontal
Connections:
- net Ropto_220: now also R17.2; no longer R2.2
- net Vadc: now also U2.4 (D34)
- net Valpha: now also U2.2 (VP)
- net Vdis1: now also U2.25 (D16/RX2)
- net Vdis2: now also U2.24 (D17/TX2)
- net Viout: now also U2.5 (D35)
- net Vzcd: now also U2.26 (D4)
- new net: R17.1, R2.2
- no-connect marks 0 -> 20
Other:
- moved on the sheet: R1, R2
